File: hw-dev-breakout/hw-dev-breakout.kicad_sch (KiCad schematic)
At the start: 30 parts, among them J101 CN7, J102 CN10, SW101 SW_Push, U101 SN65HVD232DR, U102 SN65HVD232DR, U103 SN65HVD232DR, U104 L7805

Commit message: pcb: Update some LCSC part numbers
Parts:
- J101, J102: LCSC Part # C18905898 -> C22373924
Changed lines of the file:
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@@
 			)
 		)
-		(property "LCSC Part #" "C18905898"
+		(property "LCSC Part #" " C22373924 "
 			(at 40.64 45.72 0)
 			(effects
@@
 			)
 		)
-		(property "LCSC Part #" "C18905898"
+		(property "LCSC Part #" " C22373924 "
 			(at 40.64 109.22 0)
 			(effects
